File: hardware/CDB/CDB.kicad_sch (KiCad schematic)
At the start: 17 parts, among them J1 Servo Motor, J2 Bateria, J3 Antena LoRa, Q1 BC547, U1 ESP32-C3, U2 RFM95W, U3 GPS, U4 BMP280, U5 GY-521

Commit message: Update CDB.kicad_sch
Parts:
- removed BZ2: Buzzer, Buzzer_Beeper:Buzzer_12x9.5RM7.6, symbol Device:Buzzer
- removed D1: 1N4007, PCM_Diode_THT_AKL:D_DO-41_SOD81_P7.62mm_Horizontal, symbol PCM_Diode_AKL:1N4007
- removed J1: Servo Motor, Connector:FanPinHeader_1x03_P2.54mm_Vertical, symbol Connector_Generic:Conn_01x03
- removed Q1: BC547, Package_TO_SOT_THT:TO-92_Inline, symbol Transistor_BJT:BC547
- removed R1: 1k, Resistor_THT:R_Axial_DIN0204_L3.6mm_D1.6mm_P5.08mm_Horizontal, symbol Device:R
- removed U5: GY-521, Library:GY-521, symbol New_Library:GY-521
- added J1: Micro_SD_Card, Connector_PinHeader_2.54mm:PinHeader_1x06_P2.54mm_Vertical, symbol Connector:Micro_SD_Card
- added U6: ICM-20602, Package_LGA:LGA-16_3x3mm_P0.5mm_LayoutBorder3x5y, symbol Sensor_Motion:ICM-20602
- U4: value BMP280 -> BME280
Connections:
- net at U2.1 (GND): now also J1.6 (VSS)
- net at C1.2, C2.2, C3.2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: now also U6.10 (GND), U6.11 (GND), U6.12 (GND), U6.13 (GND), U6.15 (GND), U6.9 (GND)
- net at C2.1, C3.1, C4.1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: now also J1.4 (VDD), U6.16 (VDD)
- net at U1.5 (GPIO5), U2.2 (MISO): now also J1.7 (DAT0)
- net at U1.6 (GPIO6), U2.3 (MOSI): now also J1.3 (CMD)
- net at U1.4 (GPIO4), U2.4 (SCK): now also J1.5 (CLK)
- net at U1.9 (GPIO9), U4.3 (SCL): now also U6.2 (SCL/SPC)
- net at U1.8 (GPIO8), U4.4 (SDA): now also U6.3 (SDA/SDI)
- net at U1.0 (GPIO0): now also J1.2 (DAT3/CD)
- no-connect marks 0 -> 1
Other:
- moved on the sheet: C3
